File: esp_thermometer/esp_thermometer.sch (EAGLE design)
At the start: 11 parts, among them U2 DS18B20

Commit message: Fertiger Schaltplan und Layout esp-thermometer
Parts:
- added C2: 1N00, rcl:C-EUC1206K
- added C3: 100n, rcl:C-EUC1206K
- added C4: 100N, rcl:C-EUC0805
- added C5: 47U0, rcl:C-EUC1210
- added C6: (no value), rcl:C-EUC1210
- added C7: 8N20, rcl:C-EUC0805
- added C8: 3N00, rcl:C-EUC0805
- added C9: 68N0, rcl:C-EUC0805
- added D1, D2: MBR0520LT, diode:MBR0520LT
- added D3: SS24FL, slqlib:SS24FL
- added JP1: (no value), jumper:JP1E
- added L1: SRN5020-220M, slqlib:SRN5020-220M
- added R10, R13, R9: 0R00, rcl:R-EU_R0805
- added R11, R15, R16, R17, R18: 10K2, rcl:R-EU_R0805
- added R12: 3K24, rcl:R-EU_R0805
- added R14: 10k2, rcl:R-EU_R0805
- added R7, R8: 1K00, rcl:R-EU_R0805
- added SV3: (no value), con-lstb:MA03-1
- added SV4: (no value), con-lsta:FE06-1
- added U3: TPS54231D, slqlib:TPS54231D
- added U4, U5: TLP183, slqlib:TLP183
- C1: value (none) -> 10N0
- R1, R2, R3: value (none) -> 0R00; device rcl:R-EU_R1206 -> rcl:R-EU_R0805
- R4, R5: value (none) -> 1K00; device rcl:R-EU_R1206 -> rcl:R-EU_R0805
- R6: value (none) -> 4K70; device rcl:R-EU_R1206 -> rcl:R-EU_R0805
- SV1: device con-lstb:MA05-1 -> con-lstb:MA04-1
- SV2: device con-lstb:MA03-1 -> con-lstb:MA08-2
Connections:
- new net +3V3: C1.1, C2.1, C5.1, L1.2, R11.2, R13.2, R4.1, R5.2, R6.2, R8.1, SV2.15, SV2.16, SV3.3, SV4.4, U1.VCC, U2.VDD
- new net ADC: SV2.13, U1.ADC
- new net CH_PD: R3.1, R8.2, U1.CH_PD
- new net CS0: U1.CS0
- new net GND: C1.2, C2.2, C5.2, C6.1, C7.2, C8.2, C9.2, D3.C, JP1.1, R12.1, R7.2, SV2.1, SV2.2, SV2.3, SV3.1, SV4.6, U1.GND, U2.GND, U3.GND, U4.EMIT, U5.C
- new net GPIO0: D2.A, R6.1, SV3.2, U1.GPIO0, U2.DQ
- new net GPIO10: SV2.10, U1.*GPIO10
- new net GPIO12: SV2.11, U1.GPIO12
- new net GPIO13: SV2.12, U1.GPIO13
- new net GPIO14: SV2.14, U1.GPIO14
- new net GPIO4: R18.2, SV2.6, U1.GPIO4
- new net GPIO5: R16.2, SV2.7, U1.GPIO5
- new net GPIO9: SV2.8, U1.*GPIO9
- new net MISO: SV2.9, U1.MISO
- new net MOSI: SV2.5, U1.MOSI
- new net N$1: R9.2, U1.GPIO16
- new net N$10: C3.1, R10.2, R3.2
- new net N$11: R15.1, SV1.4
- new net N$12: SV1.3, U4.C
- new net N$13: R11.1, R12.2, U3.VSENSE
- new net N$14: R17.1, SV1.2
- new net N$15: C7.1, U3.SS
- new net N$16: C8.1, R14.1
- new net N$17: C9.1, R14.2, U3.COMP
- new net N$18: R17.2, U5.COL
- new net N$19: R16.1, U4.COL
- new net N$2: C4.1, U3.BOOT
- new net N$20: SV1.1, U5.EMIT
- new net N$21: R18.1, U5.A
- new net N$3: R5.1, U1.GPIO2
- new net N$4: R1.2, SV4.2
- new net N$5: R7.1, U1.GPIO15
- new net N$6: R15.2, U4.A
- new net N$7: R2.2, SV4.3
- new net N$8: D1.C, SV4.1
- new net N$9: C3.2, D1.A, D2.C
- new net PH: C4.2, D3.A, L1.1, U3.PH
- new net RESET: R10.1, R4.2, R9.1, U1.RESET
- new net RX: R2.1, U1.RX
- new net SCLK: SV2.4, U1.SCLK
- new net TX: R1.1, U1.TX
- new net VDD: C6.2, JP1.2, R13.1, U3.VIN
Other:
- moved on the sheet: C1, R1, R2, R3, R4, R5, R6, U1, U2
